Commit message: added no payload sensor version

File: urdf/anymal_with_inspection_payload.urdf (robot description, URDF)
Before this commit: robot anymal, 87 links, 86 joints
Links:
- added link inspection_payload_camera
- added link inspection_payload_camera_default
- added link inspection_payload_head
- added link inspection_payload_light
- added link inspection_payload_microphone
- added link inspection_payload_mount, mass 0.21580; collision box size=0.16 0.135 0.015; visual mesh filename=package://anymal_d_simple_description/meshes/mount.dae scale=1 1 1
- added link inspection_payload_pan, mass 3.18886; collision box size=0.18 0.24 0.21; visual mesh filename=package://anymal_d_simple_description/meshes/pan.dae scale=1 1 1
- added link inspection_payload_thermal_camera
- added link inspection_payload_tilt, mass 2.084; visual mesh filename=package://anymal_d_simple_description/meshes/tilt.dae scale=1 1 1
Joints:
- added joint base_to_inspection_payload_mount: type fixed, parent base, child inspection_payload_mount, origin xyz=0.14253 0.0 0.092 rpy=0 0 0
- added joint inspection_payload_head_to_camera: type fixed, parent inspection_payload_head, child inspection_payload_camera, origin xyz=0.055 -0.023 0.031 rpy=-1.57079633 0 -1.57079633
- added joint inspection_payload_head_to_light: type fixed, parent inspection_payload_head, child inspection_payload_light, origin xyz=0.05495 0.03000 0.03116 rpy=-1.57079633 0 -1.57079633
- added joint inspection_payload_head_to_microphone: type fixed, parent inspection_payload_head, child inspection_payload_microphone, origin xyz=0.06840 0.02300 -0.03000 rpy=-1.57079633 0 -1.57079633
- added joint inspection_payload_head_to_thermal_camera: type fixed, parent inspection_payload_head, child inspection_payload_thermal_camera, origin xyz=0.06840 -0.02300 -0.03000 rpy=-1.57079633 0 -1.57079633
- added joint inspection_payload_mount_to_camera_default: type fixed, parent inspection_payload_mount, child inspection_payload_camera_default, origin xyz=0.0 0.0 0.175 rpy=0 0 0
- added joint inspection_payload_mount_to_pan: type revolute, parent inspection_payload_mount, child inspection_payload_pan, origin xyz=0 0 0.023 rpy=0 0 0, axis 0 0 1, limit lower=-2.6 upper=2.6 effort=20 velocity=2
- added joint inspection_payload_pan_to_tilt: type revolute, parent inspection_payload_pan, child inspection_payload_tilt, origin xyz=0.03 0 0.152 rpy=0 0 0, axis 0 1 0, limit lower=-1.570796 upper=1.570796 effort=20 velocity=2
- added joint inspection_payload_tilt_to_head: type fixed, parent inspection_payload_tilt, child inspection_payload_head, origin xyz=0.0 0.0 0.0 rpy=0 0 0
